Commit message: add

File: my_robot_description/urdf/my_robot.urdf.xacro (robot description, xacro)
@@ -1,4 +1,9 @@
 <?xml version="1.0"?>
-<robot name="my_robot">
+<robot name="my_robot" xmlns:xacro="https://www.ros.org/wiki/xacro">
+    <xacro:property name="base_length" value="0.6"/>
+    <xacro:property name="base_width" value="0.4"/>
+    <xacro:property name="base_height" value="0.2"/>
+    <xacro:property name="wheel_radius" value="0.1"/>
+    <xacro:property name="wheel_length" value="0.05"/>
     <material name="blue">
         <color rgba="0 0 0.5 1"/>
@@ -10,16 +15,29 @@
         <visual>
             <geometry>
-                <box size="0.6 0.4 0.2" />
+                <box size="${base_length} ${base_width} ${base_height}" />
             </geometry>
-            <origin xyz="0 0 0.1" rpy="0 0 0" />
+            <origin xyz="0 0 ${base_height/2.0}" rpy="0 0 0" />
             <material name="blue"/>
         </visual>
     </link>
-    <link name="right_wheel_link">
+    <xacro:macro name="wheel_link" params="prefix">
+        <link name="${prefix}_wheel_link">
+            <visual>
+                <geometry>
+                    <cylinder radius="${wheel_radius}" length="${wheel_length}"/>
+                </geometry>
+                <origin xyz="0 0 0" rpy="${pi/2.0} 0 0" />
+                <material name="grey" />
+            </visual>
+        </link>
+    </xacro:macro>
+    <xacro:wheel_link prefix="right"/>
+    <xacro:wheel_link prefix="left"/>
+    <!-- <link name="right_wheel_link">
         <visual>
             <geometry>
-                <cylinder radius="0.1" length="0.05"/>
+                <cylinder radius="${wheel_radius}" length="${wheel_length}"/>
             </geometry>
-            <origin xyz="0 0 0" rpy="1.57 0 0" />
+            <origin xyz="0 0 0" rpy="${pi/2.0} 0 0" />
             <material name="grey" />
         </visual>
@@ -28,14 +46,14 @@
         <visual>
             <geometry>
-                <cylinder radius="0.1" length="0.05"/>
+                <cylinder radius="${wheel_radius}" length="${wheel_length}"/>
             </geometry>
-            <origin xyz="0 0 0" rpy="1.57 0 0" />
+            <origin xyz="0 0 0" rpy="${pi/2.0} 0 0" />
             <material name="grey" />
         </visual>
-    </link>
+    </link> -->
     <link name="caster_wheel_link">
         <visual>
             <geometry>
-                <sphere radius="0.05"/>
+                <sphere radius="${wheel_radius/2.0}"/>
             </geometry>
             <origin xyz="0 0 0" rpy="0 0 0"/>
@@ -47,5 +65,5 @@
         <parent link="base_link"/>
         <child link="right_wheel_link"/>
-        <origin xyz="-0.15 -0.225 0" rpy="0 0 0"/>
+        <origin xyz="${-base_length/4.0} ${-(base_width/2.0+wheel_length/2.0)} 0" rpy="0 0 0"/>
         <axis xyz="0 1 0"/>
     </joint>
@@ -53,5 +71,5 @@
         <parent link="base_link"/>
         <child link="left_wheel_link"/>
-        <origin xyz="-0.15 0.225 0" rpy="0 0 0"/>
+        <origin xyz="${-base_length/4.0} ${(base_width/2.0+wheel_length/2.0)} 0" rpy="0 0 0"/>
         <axis xyz="0 1 0"/>
     </joint>
@@ -59,10 +77,10 @@
         <parent link="base_link"/>
         <child link="caster_wheel_link"/>
-        <origin xyz="0.2 0 -0.05" rpy="0 0 0"/>
+        <origin xyz="${base_length/3.0} 0 ${-wheel_radius/2.0}" rpy="0 0 0"/>
     </joint>
     <joint name="base_footprint_link" type="fixed">
         <parent link="base_footprint"/>
         <child link="base_link"/>
-        <origin xyz="0 0 0.1" rpy="0 0 0"/>
+        <origin xyz="0 0 ${wheel_radius}" rpy="0 0 0"/>
     </joint>
 </robot>

Commit message: add

File: my_robot_description/urdf/my_robot.urdf.xacro (robot description, xacro)
@@ -1,86 +1,5 @@
 <?xml version="1.0"?>
 <robot name="my_robot" xmlns:xacro="https://www.ros.org/wiki/xacro">
-    <xacro:property name="base_length" value="0.6"/>
-    <xacro:property name="base_width" value="0.4"/>
-    <xacro:property name="base_height" value="0.2"/>
-    <xacro:property name="wheel_radius" value="0.1"/>
-    <xacro:property name="wheel_length" value="0.05"/>
-    <material name="blue">
-        <color rgba="0 0 0.5 1"/>
-    </material>
-    <material name="grey">
-        <color rgba="0.5 0.5 0.5 1"/>
-    </material>
-    <link name="base_link">
-        <visual>
-            <geometry>
-                <box size="${base_length} ${base_width} ${base_height}" />
-            </geometry>
-            <origin xyz="0 0 ${base_height/2.0}" rpy="0 0 0" />
-            <material name="blue"/>
-        </visual>
-    </link>
-    <xacro:macro name="wheel_link" params="prefix">
-        <link name="${prefix}_wheel_link">
-            <visual>
-                <geometry>
-                    <cylinder radius="${wheel_radius}" length="${wheel_length}"/>
-                </geometry>
-                <origin xyz="0 0 0" rpy="${pi/2.0} 0 0" />
-                <material name="grey" />
-            </visual>
-        </link>
-    </xacro:macro>
-    <xacro:wheel_link prefix="right"/>
-    <xacro:wheel_link prefix="left"/>
-    <!-- <link name="right_wheel_link">
-        <visual>
-            <geometry>
-                <cylinder radius="${wheel_radius}" length="${wheel_length}"/>
-            </geometry>
-            <origin xyz="0 0 0" rpy="${pi/2.0} 0 0" />
-            <material name="grey" />
-        </visual>
-    </link>
-    <link name="left_wheel_link">
-        <visual>
-            <geometry>
-                <cylinder radius="${wheel_radius}" length="${wheel_length}"/>
-            </geometry>
-            <origin xyz="0 0 0" rpy="${pi/2.0} 0 0" />
-            <material name="grey" />
-        </visual>
-    </link> -->
-    <link name="caster_wheel_link">
-        <visual>
-            <geometry>
-                <sphere radius="${wheel_radius/2.0}"/>
-            </geometry>
-            <origin xyz="0 0 0" rpy="0 0 0"/>
-            <material name="grey"/>
-        </visual>
-    </link>
-    <link name="base_footprint"/>
-    <joint name="base_right_wheel_joint" type="continuous">
-        <parent link="base_link"/>
-        <child link="right_wheel_link"/>
-        <origin xyz="${-base_length/4.0} ${-(base_width/2.0+wheel_length/2.0)} 0" rpy="0 0 0"/>
-        <axis xyz="0 1 0"/>
-    </joint>
-    <joint name="base_left_wheel_joint" type="continuous">
-        <parent link="base_link"/>
-        <child link="left_wheel_link"/>
-        <origin xyz="${-base_length/4.0} ${(base_width/2.0+wheel_length/2.0)} 0" rpy="0 0 0"/>
-        <axis xyz="0 1 0"/>
-    </joint>
-    <joint name="base_caster_wheel_link" type="fixed">
-        <parent link="base_link"/>
-        <child link="caster_wheel_link"/>
-        <origin xyz="${base_length/3.0} 0 ${-wheel_radius/2.0}" rpy="0 0 0"/>
-    </joint>
-    <joint name="base_footprint_link" type="fixed">
-        <parent link="base_footprint"/>
-        <child link="base_link"/>
-        <origin xyz="0 0 ${wheel_radius}" rpy="0 0 0"/>
-    </joint>
+    <xacro:include filename="common_properties.xacro"/>
+    <xacro:include filename="mobile_base.xacro"/>
 </robot>
