Commit message: add

File: my_robot_description/urdf/common_properties.xacro (robot description, xacro)
@@ -1,9 +1,36 @@
 <?xml version="1.0"?>
-<robot xmlns:xacro="https://www.ros.org/wiki/xacro">
+<robot xmlns:xacro="http://www.ros.org/wiki/xacro">
     <material name="blue">
-        <color rgba="0 0 0.5 1"/>
+        <color rgba="0 0 0.5 1" />
     </material>
     <material name="grey">
-        <color rgba="0.5 0.5 0.5 1"/>
+        <color rgba="0.5 0.5 0.5 1" />
     </material>
+    <xacro:macro name="box_inertia" params="m l w h xyz rpy">
+        <inertial>
+            <origin xyz="${xyz}" rpy="${rpy}" />
+            <mass value="${m}" />
+            <inertia ixx="${(m/12) * (h*h + l*l)}" ixy="0" ixz="0"
+                     iyy="${(m/12) * (w*w + l*l)}" iyz="0"
+                     izz="${(m/12) * (w*w + h*h)}" />
+        </inertial>
+    </xacro:macro>
+    <xacro:macro name="cylinder_inertia" params="m r h xyz rpy">
+        <inertial>
+            <origin xyz="${xyz}" rpy="${rpy}" />
+            <mass value="${m}" />
+            <inertia ixx="${(m/12) * (3*r*r + h*h)}" ixy="0" ixz="0"
+                     iyy="${(m/12) * (3*r*r + h*h)}" iyz="0"
+                     izz="${(m/2) * (r*r)}" />
+        </inertial>
+    </xacro:macro>
+    <xacro:macro name="sphere_inertia" params="m r xyz rpy">
+        <inertial>
+            <origin xyz="${xyz}" rpy="${rpy}" />
+            <mass value="${m}" />
+            <inertia ixx="${(2/5) * m * r * r}" ixy="0" ixz="0"
+                     iyy="${(2/5) * m * r * r}" iyz="0"
+                     izz="${(2/5) * m * r * r}" />
+        </inertial>
+    </xacro:macro>
 </robot>

File: my_robot_description/urdf/mobile_base.xacro (robot description, xacro)
@@ -1,9 +1,10 @@
 <?xml version="1.0"?>
-<robot xmlns:xacro="https://www.ros.org/wiki/xacro">
-    <xacro:property name="base_length" value="0.6"/>
-    <xacro:property name="base_width" value="0.4"/>
-    <xacro:property name="base_height" value="0.2"/>
-    <xacro:property name="wheel_radius" value="0.1"/>
-    <xacro:property name="wheel_length" value="0.05"/>
+<robot xmlns:xacro="http://www.ros.org/wiki/xacro">
+    <xacro:property name="base_length" value="0.6" />
+    <xacro:property name="base_width" value="0.4" />
+    <xacro:property name="base_height" value="0.2" />
+    <xacro:property name="wheel_radius" value="0.1" />
+    <xacro:property name="wheel_length" value="0.05" />
+    <link name="base_footprint" />
     <link name="base_link">
         <visual>
@@ -11,7 +12,9 @@
                 <box size="${base_length} ${base_width} ${base_height}" />
             </geometry>
-            <origin xyz="0 0 ${base_height/2.0}" rpy="0 0 0" />
-            <material name="blue"/>
+            <origin xyz="0 0 ${base_height / 2.0}" rpy="0 0 0" />
+            <material name="blue" />
         </visual>
+        <xacro:box_inertia m="5.0" l="${base_length}" w="${base_width}" h="${base_height}"
+                           xyz="0 0 ${base_height / 2.0}" rpy="0 0 0" />
     </link>
     <xacro:macro name="wheel_link" params="prefix">
@@ -19,44 +22,47 @@
             <visual>
                 <geometry>
-                    <cylinder radius="${wheel_radius}" length="${wheel_length}"/>
+                    <cylinder radius="${wheel_radius}" length="${wheel_length}" />
                 </geometry>
-                <origin xyz="0 0 0" rpy="${pi/2.0} 0 0" />
+                <origin xyz="0 0 0" rpy="${pi / 2.0} 0 0" />
                 <material name="grey" />
             </visual>
+            <xacro:cylinder_inertia m="1.0" r="${wheel_radius}" h="${wheel_length}"
+                                    xyz="0 0 0" rpy="${pi / 2.0} 0 0" />
         </link>
     </xacro:macro>
-    <xacro:wheel_link prefix="right"/>
-    <xacro:wheel_link prefix="left"/>
+    <xacro:wheel_link prefix="right" />
+    <xacro:wheel_link prefix="left" />
     <link name="caster_wheel_link">
         <visual>
             <geometry>
-                <sphere radius="${wheel_radius/2.0}"/>
+                <sphere radius="${wheel_radius / 2.0}" />
             </geometry>
-            <origin xyz="0 0 0" rpy="0 0 0"/>
-            <material name="grey"/>
+            <origin xyz="0 0 0" rpy="0 0 0" />
+            <material name="grey" />
         </visual>
+        <xacro:sphere_inertia m="0.5" r="${wheel_radius / 2.0}"
+                              xyz="0 0 0" rpy="0 0 0" />
     </link>
-    <link name="base_footprint"/>
+    <joint name="base_joint" type="fixed">
+        <parent link="base_footprint" />
+        <child link="base_link" />
+        <origin xyz="0 0 ${wheel_radius}" rpy="0 0 0"/>
+    </joint>
     <joint name="base_right_wheel_joint" type="continuous">
-        <parent link="base_link"/>
-        <child link="right_wheel_link"/>
-        <origin xyz="${-base_length/4.0} ${-(base_width/2.0+wheel_length/2.0)} 0" rpy="0 0 0"/>
-        <axis xyz="0 1 0"/>
+        <parent link="base_link" />
+        <child link="right_wheel_link" />
+        <origin xyz="${-base_length / 4.0} ${-(base_width + wheel_length) / 2.0} 0" rpy="0 0 0" />
+        <axis xyz="0 1 0" />
     </joint>
     <joint name="base_left_wheel_joint" type="continuous">
-        <parent link="base_link"/>
-        <child link="left_wheel_link"/>
-        <origin xyz="${-base_length/4.0} ${(base_width/2.0+wheel_length/2.0)} 0" rpy="0 0 0"/>
-        <axis xyz="0 1 0"/>
+        <parent link="base_link" />
+        <child link="left_wheel_link" />
+        <origin xyz="${-base_length / 4.0} ${(base_width + wheel_length) / 2.0} 0" rpy="0 0 0" />
+        <axis xyz="0 1 0" />
     </joint>
-    <joint name="base_caster_wheel_link" type="fixed">
-        <parent link="base_link"/>
-        <child link="caster_wheel_link"/>
-        <origin xyz="${base_length/3.0} 0 ${-wheel_radius/2.0}" rpy="0 0 0"/>
-    </joint>
-    <joint name="base_footprint_link" type="fixed">
-        <parent link="base_footprint"/>
-        <child link="base_link"/>
-        <origin xyz="0 0 ${wheel_radius}" rpy="0 0 0"/>
+    <joint name="base_caster_wheel_joint" type="fixed">
+        <parent link="base_link" />
+        <child link="caster_wheel_link" />
+        <origin xyz="${base_length / 3.0} 0 ${-wheel_radius / 2.0}" rpy="0 0 0" />
     </joint>
 </robot>

Commit message: add

File: my_robot_description/urdf/common_properties.xacro (robot description, xacro)
@@ -6,4 +6,7 @@
     <material name="grey">
         <color rgba="0.5 0.5 0.5 1" />
+    </material>
+    <material name="orange">
+        <color rgba="1.0 0.5 0 1">
     </material>
     <xacro:macro name="box_inertia" params="m l w h xyz rpy">

File: my_robot_description/urdf/mobile_base.xacro (robot description, xacro)
@@ -15,5 +15,11 @@
             <material name="blue" />
         </visual>
-        <xacro:box_inertia m="5.0" l="${base_length}" w="${base_width}" h="${base_height}"
+        <collision>
+            <geometry>
+                <box size="${base_length} ${base_width} ${base_height}" />
+            </geometry>
+            <origin xyz="0 0 ${base_height / 2.0}" rpy="0 0 0" />
+        </collision>
+        <xacro:box_inertia m="5.0" l="${2*base_length}" w="${2*base_width}" h="${2*base_height}"
                            xyz="0 0 ${base_height / 2.0}" rpy="0 0 0" />
     </link>
@@ -27,5 +33,11 @@
                 <material name="grey" />
             </visual>
-            <xacro:cylinder_inertia m="1.0" r="${wheel_radius}" h="${wheel_length}"
+            <collision>
+                <geometry>
+                    <cylinder radius="${wheel_radius}" length="${wheel_length}" />
+                </geometry>
+                <origin xyz="0 0 0" rpy="${pi / 2.0} 0 0" />
+            </collision>
+            <xacro:cylinder_inertia m="1.0" r="${2*wheel_radius}" h="${2*wheel_length}"
                                     xyz="0 0 0" rpy="${pi / 2.0} 0 0" />
         </link>
@@ -41,5 +53,11 @@
             <material name="grey" />
         </visual>
-        <xacro:sphere_inertia m="0.5" r="${wheel_radius / 2.0}"
+        <collision>
+            <geometry>
+                <sphere radius="${wheel_radius / 2.0}" />
+            </geometry>
+            <origin xyz="0 0 0" rpy="0 0 0" />
+        </collision>
+        <xacro:sphere_inertia m="0.5" r="${2*wheel_radius / 2.0}"
                               xyz="0 0 0" rpy="0 0 0" />
     </link>

File: my_robot_description/urdf/my_robot.urdf.xacro (robot description, xacro)
@@ -3,3 +3,5 @@
     <xacro:include filename="common_properties.xacro"/>
     <xacro:include filename="mobile_base.xacro"/>
+    <xacro:include filename="mobile_base_gazebo.xacro"/>
+    <xacro:include filename="camera.xacro"/>
 </robot>
